File: Camera_PCB/Camera_PCB.kicad_sch (KiCad schematic)
At the start: 1 part, among them U1 V3s-eLQFP128

Commit message: Started PCB
Connections:
- net AGND: no longer names the net of U1.116 (AGND)
- net AVCC: no longer names the net of U1.115 (AVCC)
- net HPVCCBP: no longer names the net of U1.123 (HPVCCBP)
- net KEYADC0: no longer names the net of U1.112 (LARDC0)
- no-connect marks 59 -> 63
Changed lines of the file:
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@@
+	)
+	(no_connect
+		(at 73.66 29.21)
 	)
 	(no_connect
@@
 	)
 	(no_connect
+		(at 91.44 29.21)
+	)
+	(no_connect
 		(at 170.18 69.85)
 	)
@@
 	)
 	(no_connect
+		(at 93.98 29.21)
+	)
+	(no_connect
 		(at 170.18 57.15)
 	)
@@
 	)
 	(no_connect
+		(at 101.6 29.21)
+	)
+	(no_connect
 		(at 35.56 130.81)
 	)
@@
 	(wire
 		(pts
-			(xy 101.6 26.67) (xy 101.6 29.21)
-		)
-		(stroke
-			(width 0)
-			(type default)
-		)
-	)
-	(wire
-		(pts
 			(xy 170.18 80.01) (xy 172.72 80.01)
 		)
@@
 	(wire
 		(pts
-			(xy 91.44 26.67) (xy 91.44 29.21)
-		)
-		(stroke
-			(width 0)
-			(type default)
-		)
-	)
-	(wire
-		(pts
 			(xy 121.92 26.67) (xy 121.92 29.21)
 		)
@@
 	(wire
 		(pts
-			(xy 73.66 26.67) (xy 73.66 29.21)
-		)
-		(stroke
-			(width 0)
-			(type default)
-		)
-	)
-	(wire
-		(pts
 			(xy 153.67 26.67) (xy 153.67 29.21)
 		)
@@
 	(wire
 		(pts
-			(xy 93.98 26.67) (xy 93.98 29.21)
-		)
-		(stroke
-			(width 0)
-			(type default)
-		)
-	)
-	(wire
-		(pts
 			(xy 35.56 123.19) (xy 33.02 123.19)
 		)
@@
 		)
 	)
-	(global_label "AVCC"
-		(shape bidirectional)
-		(at 93.98 26.67 90)
-		(fields_autoplaced yes)
-		(effects
-			(font
-				(size 1.27 1.27)
-			)
-			(justify left)
-		)
-		(property "Intersheetrefs" "${INTERSHEET_REFS}"
-			(at 93.98 17.8563 90)
-			(effects
-				(font
-					(size 1.27 1.27)
-				)
-				(justify left)
-				(hide yes)
-			)
-		)
-	)
 	(global_label "VCC-USB"
 		(shape bidirectional)
@@
 		)
 	)
-	(global_label "AGND"
-		(shape bidirectional)
-		(at 91.44 26.67 90)
-		(fields_autoplaced yes)
-		(effects
-			(font
-				(size 1.27 1.27)
-			)
-			(justify left)
-		)
-		(property "Intersheetrefs" "${INTERSHEET_REFS}"
-			(at 91.44 17.6144 90)
-			(effects
-				(font
-					(size 1.27 1.27)
-				)
-				(justify left)
-				(hide yes)
-			)
-		)
-	)
 	(global_label "VDD-SYS"
 		(shape bidirectional)
@@
 		)
 	)
-	(global_label "KEYADC0"
-		(shape bidirectional)
-		(at 101.6 26.67 90)
-		(fields_autoplaced yes)
-		(effects
-			(font
-				(size 1.27 1.27)
-			)
-			(justify left)
-		)
-		(property "Intersheetrefs" "${INTERSHEET_REFS}"
-			(at 101.6 14.2278 90)
-			(effects
-				(font
-					(size 1.27 1.27)
-				)
-				(justify left)
-				(hide yes)
-			)
-		)
-	)
 	(global_label "SDC0_D1"
 		(shape bidirectional)
@@
 			(effects
 				(font
-					(size 1.27 1.27)
-				)
-				(justify left)
-				(hide yes)
-			)
-		)
-	)
-	(global_label "HPVCCBP"
-		(shape bidirectional)
-		(at 73.66 26.67 90)
-		(fields_autoplaced yes)
-		(effects
-			(font
-				(size 1.27 1.27)
-			)
-			(justify left)
-		)
-		(property "Intersheetrefs" "${INTERSHEET_REFS}"
-			(at 73.66 13.8044 90)
-			(effects
-				(font
