File: Camera_PCB/V3s.kicad_sch (KiCad schematic)
At the start: 1 part, among them U2 V3s-eLQFP128

Commit message: Camera PCB Schematic review 1
Connections:
- net UART2_TX: now reaches U2.39 (PB0)
- net UART2_RX: now reaches U2.40 (PB1)
- net IRQ: now reaches U2.42 (PB3)
- net CAM_EN0: now reaches U2.44 (PB5)
- net TWI0_SCK: now reaches U2.45 (PB6)
- net TWI0_SDA: now reaches U2.46 (PB7)
- net UART0_TX: now reaches U2.48 (PB8)
- net UART0_RX: now reaches U2.49 (PB9)
- no-connect marks 63 -> 55
Other:
- note added: "Expose UART 0 for System UART"
- note added: "Expose UART 2 for backup UART"
- note removed: "P39, P40 UART2 Pins"
- note removed: "P41 - P44 MISC Pins"
- note removed: "P45, P46, P48, P49 are 2 TWI lines"
