File: Camera_PCB/CameraPCB.kicad_pcb (KiCad board)
At the start: 6 copper layers, 65.6 x 55 mm, 173 parts, among them J1 MIPI-CSI2, J2 USB_A, J3 SDA, J4 UART_0, J5 UART_2, J6 USB_C_Receptacle_PowerOnly_6P, SW1 PWR, SW2 RST, U1 AXP203, U2 V3s-eLQFP128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

Commit message: resized vias to 0.2/0.45mm
Routing:
- net GND: track 20.7 -> 21.8 mm
- net PWREN: track 68.7 -> 69.3 mm
