File: Camera_PCB/3V3_5V0.kicad_sch (KiCad schematic)
At the start: 22 parts

Commit message: Thorough Camera PCB Review by Jack
Parts:
- removed TPS63020, TPS63021: ~, BackupCamCustomParts:IC_TPS63020DSJT, symbol Senior:TPS63020
- added TP21: 5V, TestPoint:TestPoint_Pad_D1.5mm, symbol Connector:TestPoint
- added TP22: 3V3, TestPoint:TestPoint_Pad_D1.5mm, symbol Connector:TestPoint
- added TP23: 3V3FB, TestPoint:TestPoint_Pad_D1.5mm, symbol Connector:TestPoint
- added TP24: 5V0FB, TestPoint:TestPoint_Pad_D1.5mm, symbol Connector:TestPoint
- added U3, U4: TPS63020, BackupCamCustomParts:IC_TPS63020DSJT, symbol custom_chips:TPS63020
Connections:
- net +3V3: now also TP22.1, U4.4 (VOUT), U4.5 (VOUT)
- net +5V: now also TP21.1, U3.4 (VOUT), U3.5 (VOUT)
- net GND: now also C66.2, C69.2, U3.13 (PS/SYNC), U3.15 (PGND), U3.2 (GND), U4.13 (PS/SYNC), U4.15 (PGND), U4.2 (GND)
- net PWREN: now also U3.12 (EN), U4.12 (EN)
- net VBAT: now also U3.10 (VIN), U3.11 (VIN), U4.10 (VIN), U4.11 (VIN)
- net at R26.2, R27.1: now also TP23.1, U4.3 (FB)
- net VIPS: now reaches C52.1
- net VIPS: now also C2.1, U3.1 (VINA), U4.1 (VINA)
- net at L2.1: now also U4.6 (L2), U4.7 (L2)
- net at L2.2: now also U4.8 (L1), U4.9 (L1)
- net at R24.2, R25.1: now also TP24.1, U3.3 (FB)
- net at L1.1: now also U3.6 (L2), U3.7 (L2)
- net at L1.2: now also U3.8 (L1), U3.9 (L1)
- new net PGOOD: U3.14 (PG), U4.14 (PG)
- no-connect marks 2 -> 0
Other:
- note added: "PG is open drain high-active power good Pulls reset low if power output unstable"
- moved on the sheet: L1, L2

Commit message: more schematic changes, added solder bridges, etc
Parts:
- added JP5, JP6: ~, Jumper:SolderJumper-2_P1.3mm_Open_Pad1.0x1.5mm, symbol Jumper:Jumper_2_Small_Bridged
Connections:
- net +3V3: now also JP6.2 (B); no longer C53.1, C64.1, C65.1, C66.1, C67.1, R26.1, TP22.1, U4.4 (VOUT), U4.5 (VOUT)
- net +5V: now also JP5.2 (B); no longer C68.1, C69.1, C70.1, C71.1, C72.1, R24.1, TP21.1, U3.4 (VOUT), U3.5 (VOUT)
- new net: C68.1, C69.1, C70.1, C71.1, C72.1, JP5.1 (A), R24.1, TP21.1, U3.4 (VOUT), U3.5 (VOUT)
- new net: C53.1, C64.1, C65.1, C66.1, C67.1, JP6.1 (A), R26.1, TP22.1, U4.4 (VOUT), U4.5 (VOUT)
Other:
- moved on the sheet: TP21, TP22
Changed lines of the file:
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@@
 	)
 	(junction
-		(at 201.93 49.53)
-		(diameter 0)
-		(color 0 0 0 0)
-	)
-	(junction
 		(at 190.5 105.41)
 		(diameter 0)
@@
 	)
 	(junction
+		(at 201.93 49.53)
+		(diameter 0)
+		(color 0 0 0 0)
+	)
+	(junction
 		(at 128.27 41.91)
 		(diameter 0)
@@
 	(wire
 		(pts
-			(xy 201.93 48.26) (xy 201.93 49.53)
+			(xy 209.55 48.26) (xy 209.55 49.53)
 		)
 		(stroke
@@
 	(wire
 		(pts
-			(xy 201.93 50.8) (xy 201.93 49.53)
-		)
-		(stroke
-			(width 0)
-			(type default)
-		)
-	)
-	(wire
-		(pts
 			(xy 138.43 49.53) (xy 140.97 49.53)
 		)
@@
 	(wire
 		(pts
-			(xy 201.93 49.53) (xy 190.5 49.53)
+			(xy 209.55 49.53) (xy 208.28 49.53)
 		)
 		(stroke
@@
 	(wire
 		(pts
-			(xy 201.93 104.14) (xy 201.93 105.41)
+			(xy 212.09 102.87) (xy 212.09 105.41)
 		)
 		(stroke
@@
 	(wire
 		(pts
+			(xy 212.09 105.41) (xy 209.55 105.41)
+		)
+		(stroke
+			(width 0)
+			(type default)
+		)
+	)
+	(wire
+		(pts
 			(xy 106.68 125.73) (xy 106.68 128.27)
 		)
@@
 	(wire
 		(pts
+			(xy 190.5 49.53) (xy 201.93 49.53)
+		)
+		(stroke
+			(width 0)
+			(type default)
+		)
+	)
+	(wire
+		(pts
 			(xy 99.06 62.23) (xy 99.06 71.12)
 		)
@@
 	(wire
 		(pts
+			(xy 204.47 105.41) (xy 201.93 105.41)
+		)
+		(stroke
+			(width 0)
+			(type default)
+		)
+	)
+	(wire
+		(pts
 			(xy 190.5 106.68) (xy 190.5 105.41)
 		)
@@
 	(wire
 		(pts
+			(xy 201.93 49.53) (xy 201.93 50.8)
+		)
+		(stroke
+			(width 0)
+			(type default)
+		)
+	)
+	(wire
+		(pts
 			(xy 99.06 118.11) (xy 99.06 127)
 		)
@@
 	(wire
 		(pts
+			(xy 203.2 49.53) (xy 201.93 49.53)
+		)
+		(stroke
+			(width 0)
+			(type default)
+		)
+	)
+	(wire
+		(pts
 			(xy 118.11 97.79) (xy 119.38 97.79)
 		)
@@
 	)
 	(symbol
+		(lib_id "Jumper:Jumper_2_Small_Bridged")
+		(at 205.74 49.53 0)
+		(unit 1)
+		(exclude_from_sim no)
+		(in_bom yes)
+		(on_board yes)
+		(dnp no)
+		(property "Reference" "JP5"
+			(at 205.7198 46.99 0)
+			(effects
+				(font
+					(size 1.27 1.27)
+				)
+			)
+		)
+		(property "Value" "~"
+			(at 205.74 46.99 0)
+			(effects
+				(font
+					(size 1.27 1.27)
+				)
+			)
+		)
+		(property "Footprint" "Jumper:SolderJumper-2_P1.3mm_Open_Pad1.0x1.5mm"
+			(at 205.74 49.53 0)
+			(effects
+				(font
+					(size 1.27 1.27)
+				)
+				(hide yes)
+			)
+		)
+		(property "Datasheet" "~"
+			(at 205.74 49.53 0)
+			(effects
+				(font
+					(size 1.27 1.27)
+				)
+				(hide yes)
+			)
+		)
+		(property "Description" "Jumper, 2-pole, small symbol, bridged"
+			(at 205.74 49.53 0)
+			(effects
+				(font
+					(size 1.27 1.27)
+				)
+				(hide yes)
+			)
+		)
+		(pin "2"
+		)
+		(pin "1"
+		)
+		(instances
+			(project "CameraPCB"
+				(path "/400c1603-202c-4359-a830-d2f0d06dd3ce/f4829b1f-636b-49a4-aa22-dc0b023f0960"
+					(reference "JP5")
+					(unit 1)
+				)
+			)
+		)
+	)
+	(symbol
 		(lib_id "power:GND")
 		(at 144.78 125.73 0)
@@
 	(symbol
 		(lib_id "power:+3V3")
-		(at 201.93 104.14 0)
+		(at 212.09 102.87 0)
 		(unit 1)
 		(exclude_from_sim no)
@@
 		(fields_autoplaced yes)
 		(property "Reference" "#PWR039"
-			(at 201.93 107.95 0)
+			(at 212.09 106.68 0)
 			(effects
 				(font
@@
 		)
 		(property "Value" "+3V3"
-			(at 201.93 99.06 0)
+			(at 212.09 97.79 0)
 			(effects
 				(font
@@
 		)
 		(property "Footprint" ""
-			(at 201.93 104.14 0)
+			(at 212.09 102.87 0)
 			(effects
 				(font
@@
 		)
 		(property "Datasheet" ""
-			(at 201.93 104.14 0)
+			(at 212.09 102.87 0)
 			(effects
 				(font
@@
 		)
 		(property "Description" "Power symbol creates a global label with name \"+3V3\""
-			(at 201.93 104.14 0)
+			(at 212.09 102.87 0)
 			(effects
 				(font
@@
 	(symbol
 		(lib_id "Connector:TestPoint")
-		(at 201.93 105.41 270)
+		(at 190.5 105.41 0)
 		(unit 1)
 		(exclude_from_sim no)
@@
 		(dnp no)
 		(property "Reference" "TP22"
-			(at 207.01 104.14 90)
+			(at 191.77 100.33 0)
 			(effects
 				(font
@@
 		)
 		(property "Value" "3V3"
-			(at 207.01 106.68 90)
+			(at 191.77 104.14 0)
 			(effects
 				(font
@@
 		)
 		(property "Footprint" "TestPoint:TestPoint_Pad_D1.5mm"
-			(at 201.93 110.49 0)
+			(at 195.58 105.41 0)
 			(effects
 				(font
@@
 		)
 		(property "Datasheet" "~"
-			(at 201.93 110.49 0)
+			(at 195.58 105.41 0)
 			(effects
 				(font
@@
 		)
 		(property "Description" "test point"
-			(at 201.93 105.41 0)
+			(at 190.5 105.41 0)
 			(effects
 				(font
@@
 	(symbol
 		(lib_id "Connector:TestPoint")
-		(at 201.93 49.53 270)
+		(at 190.5 49.53 0)
 		(unit 1)
 		(exclude_from_sim no)
@@
 		(dnp no)
 		(property "Reference" "TP21"
-			(at 207.01 48.26 90)
+			(at 191.77 44.45 0)
 			(effects
 				(font
@@
 		)
 		(property "Value" "5V"
-			(at 207.01 50.8 90)
+			(at 191.77 48.26 0)
 			(effects
 				(font
@@
 		)
 		(property "Footprint" "TestPoint:TestPoint_Pad_D1.5mm"
-			(at 201.93 54.61 0)
+			(at 195.58 49.53 0)
 			(effects
 				(font
@@
 		)
 		(property "Datasheet" "~"
-			(at 201.93 54.61 0)
+			(at 195.58 49.53 0)
 			(effects
 				(font
@@
 		)
 		(property "Description" "test point"
-			(at 201.93 49.53 0)
+			(at 190.5 49.53 0)
 			(effects
 				(font
@@
 	(symbol
 		(lib_id "power:+5V")
-		(at 201.93 48.26 0)
+		(at 209.55 48.26 0)
 		(unit 1)
 		(exclude_from_sim no)
@@
 		(fields_autoplaced yes)
 		(property "Reference" "#PWR046"
-			(at 201.93 52.07 0)
+			(at 209.55 52.07 0)
 			(effects
 				(font
@@
 		)
 		(property "Value" "+5V"
-			(at 201.93 43.18 0)
+			(at 209.55 43.18 0)
 			(effects
 				(font
@@
 		)
 		(property "Footprint" ""
-			(at 201.93 48.26 0)
+			(at 209.55 48.26 0)
 			(effects
 				(font
@@
 		)
 		(property "Datasheet" ""
-			(at 201.93 48.26 0)
+			(at 209.55 48.26 0)
 			(effects
 				(font
@@
 		)
 		(property "Description" "Power symbol creates a global label with name \"+5V\""
-			(at 201.93 48.26 0)
+			(at 209.55 48.26 0)
 			(effects
 				(font
@@
 	)
 	(symbol
+		(lib_id "Jumper:Jumper_2_Small_Bridged")
+		(at 207.01 105.41 0)
+		(unit 1)
+		(exclude_from_sim no)
+		(in_bom yes)
+		(on_board yes)
+		(dnp no)
+		(property "Reference" "JP6"
+			(at 207.1648 102.87 0)
+			(effects
+				(font
+					(size 1.27 1.27)
+				)
+			)
+		)
+		(property "Value" "~"
+			(at 207.01 102.87 0)
+			(effects
+				(font
+					(size 1.27 1.27)
+				)
+			)
+		)
+		(property "Footprint" "Jumper:SolderJumper-2_P1.3mm_Open_Pad1.0x1.5mm"
+			(at 207.01 105.41 0)
+			(effects
+				(font
+					(size 1.27 1.27)
+				)
+				(hide yes)
+			)
+		)
+		(property "Datasheet" "~"
+			(at 207.01 105.41 0)
+			(effects
+				(font
+					(size 1.27 1.27)
+				)
+				(hide yes)
+			)
+		)
+		(property "Description" "Jumper, 2-pole, small symbol, bridged"
+			(at 207.01 105.41 0)
+			(effects
+				(font
+					(size 1.27 1.27)
+				)
+				(hide yes)
+			)
+		)
+		(pin "2"
+		)
+		(pin "1"
+		)
+		(instances
+			(project "CameraPCB"
+				(path "/400c1603-202c-4359-a830-d2f0d06dd3ce/f4829b1f-636b-49a4-aa22-dc0b023f0960"
+					(reference "JP6")
+					(unit 1)
+				)
+			)
+		)
+	)
+	(symbol
 		(lib_id "custom_chips:VIPS")
 		(at 106.68 118.11 0)
@@
 				)
 				(justify left)
-				(hide yes)
 			)
 		)
@@
 				)
 				(justify left)
-				(hide yes)
 			)
 		)

Commit message: PCB commit before reorganizing
Changed lines of the file:
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@@
 				)
 				(justify left)
-				(hide yes)
 			)
 		)
@@
 				)
 				(justify left)
-				(hide yes)
 			)
 		)

Commit message: updated bom for order
Parts:
- TP21, TP22, TP23, TP24: now left out of the parts list
Changed lines of the file:
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@@
 		(unit 1)
 		(exclude_from_sim no)
-		(in_bom yes)
+		(in_bom no)
 		(on_board yes)
 		(dnp no)
@@
 		(unit 1)
 		(exclude_from_sim no)
-		(in_bom yes)
+		(in_bom no)
 		(on_board yes)
 		(dnp no)
@@
 		(unit 1)
 		(exclude_from_sim no)
-		(in_bom yes)
+		(in_bom no)
 		(on_board yes)
 		(dnp no)
@@
 		(unit 1)
 		(exclude_from_sim no)
-		(in_bom yes)
-		(on_board yes)
-		(dnp no)
+		(in_bom no)
+		(on_board yes)
+		(dnp no)
