File: Camera_PCB/CSI_USB_SD_OSC.kicad_sch (KiCad schematic)
At the start: 23 parts, among them J1 MIPI-CSI2, J2 USB_A, J3 SDA, J4 UART_0, J5 UART_2, Y2 32.768kHz XTAL, Y4 24MHz XTAL

Commit message: Thorough Camera PCB Review by Jack
Parts:
- added TP25: CSCK, TestPoint:TestPoint_Pad_D1.5mm, symbol Connector:TestPoint
- added TP26: CSDA, TestPoint:TestPoint_Pad_D1.5mm, symbol Connector:TestPoint
- added TP27: CEN, TestPoint:TestPoint_Pad_D1.5mm, symbol Connector:TestPoint
- J1: symbol Connector_Generic_MountingPin:Conn_01x15_MountingPin_1 -> Connector_Generic_MountingPin:Conn_01x15_MountingPin
Connections:
- net +3.3V is gone; now on net +3V3: C34.1, J3.4 (VDD), R2.1, R3.1, R4.1, R5.1, R6.1
- net CAM_EN0: now also TP27.1
- net CSI_SCK: now also TP25.1
- net CSI_SDA: now also TP26.1
- net GND: now also J1.MP, J3.S1, J3.S2
- no-connect marks 1 -> 3

Commit message: PCB commit before reorganizing
Parts:
- added R31: 4.7k, Resistor_SMD:R_0603_1608Metric_Pad0.98x0.95mm_HandSolder, symbol Device:R_US
Connections:
- net +3V3: now also R31.1
- net CAM_EN0: now also R31.2
- net GND: now also Y2.2
- net X32KOUT: no longer Y2.2
Other:
- moved on the sheet: R13, TP26, TP27

Commit message: updated bom for order
Parts:
- TP25, TP26, TP27: now left out of the parts list
Changed lines of the file:
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@@
 		(unit 1)
 		(exclude_from_sim no)
-		(in_bom yes)
+		(in_bom no)
 		(on_board yes)
 		(dnp no)
@@
 		(unit 1)
 		(exclude_from_sim no)
-		(in_bom yes)
+		(in_bom no)
 		(on_board yes)
 		(dnp no)
@@
 		(unit 1)
 		(exclude_from_sim no)
-		(in_bom yes)
+		(in_bom no)
 		(on_board yes)
 		(dnp no)
@@
 			)
 		)
-		(property "Datasheet" "~"
+		(property "Datasheet" "https://search.murata.co.jp/Ceramy/image/img/A01X/G101/ENG/GCM188R71E105KA64-04A.pdf"
 			(at 176.53 86.36 0)
 			(effects
