File: Power/BatteryPower.kicad_sch (KiCad schematic)
At the start: 18 parts, among them J1 USB_C_Receptacle_PowerOnly_6P, Q2 AO3400A, Q3 AO3400A, U1 BQ297xy, U2 TPS63000

Commit message: restructuring main branch to have power schematic in power directory
Parts:
- added BT2: Battery_Cell, symbol Device:Battery_Cell
- added C10, C11, C12, C13, C14, C15, C16, C17, C18, C19, C20, C21, C4, C5, C6, C7, C8, C9: C, symbol Device:C
- added D1, D2: D_Schottky_Dual_CommonAnode_KAK_Split, symbol Device:D_Schottky_Dual_CommonAnode_KAK_Split
- added D3: LED, symbol Device:LED
- added L2, L3, L4: L, symbol Device:L
- added R10, R11, R12, R13, R8, R9: R, symbol Device:R
- added SW1: SW_Push, symbol Switch:SW_Push
Connections:
- net GND: now also AXP203.11 (LD04), AXP203.14 (VIN3), AXP203.22 (AGND), AXP203.27 (LDO1SET), AXP203.46 (PGND1), AXP203.49 (EP), AXP203.9 (PGND2), BT2.2 (-), C10.1, C11.1, C12.2, C13.1, C14.2, C15.2, C16.2, C17.2, C18.2, C19.2, C20.2, C21.1, C4.1, C5.2, C6.2, C7.2, C8.1, C9.1, D1.2 (A), D2.1 (K), D3.1 (K), R11.1, R8.1, SW1.1
- net IPSOUT AXP: now reaches C3.1, U2.4 (VIN)
- net V3s: now reaches AXP203.1 (SDA)
- net V3s: now also AXP203.2 (SCK)
- net DCDC2: now reaches AXP203.10 (DCDC2)
- net DCDC2: now also C15.1, C16.1, L3.2
- net at AXP203.12 (LD02): now also C21.2
- net at AXP203.15 (LX3): now also L4.1
- net at AXP203.16 (PGND3): now also C20.1
- net DCDC3: now reaches AXP203.17 (DCDC3)
- net DCDC3: now also C18.1, C19.1, L4.2
- net EN BB: now reaches AXP203.20 (EXTEN)
- net ISPOUT: now reaches AXP203.21 (APS)
- net ISPOUT: now also C9.2
- net at AXP203.23 (BIAS): now also R11.2
- net at AXP203.24 (VREF): now also C10.2
- net at AXP203.26 (VINT): now also C8.2
- net VBUS USBC: now reaches AXP203.31 (VBUS)
- net VBUS USBC: now also D2.2 (A), R9.1
- net VIN BB: now reaches AXP203.34 (IPSOUT)
- net VIN BB: now also AXP203.35 (IPSOUT), C5.1, C6.1
- net at AXP203.36 (CHGLED): now also R10.2
- net at AXP203.37 (TS): now also R8.2
- net at AXP203.38 (BAT): now also AXP203.39 (BAT), BT2.1 (+), C4.2, D1.1 (K)
- net BAT: now reaches AXP203.42 (BATSENSE)
- net BAT: now also C13.2, R13.1
- net at AXP203.43 (CHSENSE): now also C12.1, L2.2, R13.2
- net at AXP203.44 (VIN1): now also C14.1
- net at AXP203.45 (LX1): now also L2.1
- net at AXP203.47 (PWRON): now also C11.2, R12.2
- net at AXP203.7 (VIN2): now also C17.1
- net at AXP203.8 (LX2): now also L3.1
- new net: C7.1, R9.2
- new net: D3.2 (A), R10.1
- new net: R12.1, SW1.2
Other:
- moved on the sheet: AXP203, J1, R1, R2
